Commit message: Adding msg

File: robot_auto/urdf/kinect.gazebo.xacro (robot description, xacro)
@@ -10,6 +10,6 @@
           <image>
             <format>B8G8R8</format>
-            <width>640</width>
-            <height>480</height>
+            <width>1280</width>
+            <height>720</height>
           </image>
           <clip>

File: robot_auto/urdf/kinect.urdf.xacro (robot description, xacro)
@@ -2,10 +2,10 @@
 <robot name="sensor_kinect" xmlns:xacro="http://ros.org/wiki/xacro">
   <!-- Propiedades para simular con gazebo  -->
-  <xacro:include filename="$(find robot_auto)/urdf/kinect.gazebo.xacro"/>
-  <xacro:property name="cam_px" value="0.0" />
+  <xacro:include filename="$(find autlab5)/urdf/kinect.gazebo.xacro"/>
+  <xacro:property name="cam_px" value="0.1" />
   <xacro:property name="cam_py" value="0" />
-  <xacro:property name="cam_pz" value="0.077" />
+  <xacro:property name="cam_pz" value="-0.03" />
   <xacro:property name="cam_or" value="0" />
-  <xacro:property name="cam_op" value="0" />
+  <xacro:property name="cam_op" value="0.30" />
   <xacro:property name="cam_oy" value="0" />
   <xacro:property name="kinect_cam_py" value="-0.0125"/>
@@ -30,23 +30,32 @@
     </joint>
     <link name="camera_link">
+      <inertial>
+        <mass value="0.064" />
+        <origin xyz="0 0 0" />
+        <inertia ixx="5.8083e-4" ixy="0" ixz="0" iyy="3.0833e-5" iyz="0" izz="5.9083e-4"/>
+      </inertial>
       <visual>
-        <origin xyz="0 0 0" rpy="0 0 ${M_PI/2}"/>
+        <origin xyz="0 0 0" rpy="0 0 0"/>
         <geometry>
-          <mesh filename="package://robot_auto/urdf/meshes/kinect.dae"/>
+          <!-- <mesh filename="package://autlab5/urdf/meshes/kinect.dae"/> -->
+          <box size="0.007 0.130 0.02" />
         </geometry>
+        <material name="DarkGrey">
+           <color rgba="0.3 0.3 0.3 1"/>
+        </material>
       </visual>
-      <collision>
+<!--       <collision>
         <origin xyz="0.0 0.0 0.0" rpy="0 0 0"/>
   	<geometry>
   	  <box size="0.07271 0.27794 0.073"/>
   	</geometry>
-      </collision>
-      <inertial>
-        <mass value="0.564" />
-        <origin xyz="0 0 0" />
-        <inertia ixx="0.003881243" ixy="0.0" ixz="0.0"
-                 iyy="0.000498940" iyz="0.0"
-                 izz="0.003879257" />
-      </inertial>
+      </collision> -->
+        <collision>
+          <origin xyz="0 0 0" rpy="0 0 0" />
+          <geometry>
+            <!--Dimensions taken from https://software.intel.com/en-us/realsense/devkit-->
+            <box size="0.007 0.130 0.02" />
+          </geometry>
+        </collision>
     </link>
     <!-- The fixed joints & links below are usually published by static_transformers launched by the OpenNi launch

File: robot_auto/urdf/robot_quadrotor_hokuyo.urdf.xacro (robot description, xacro)
@@ -6,7 +6,15 @@
     <!-- Instantiate quadrotor_base_macro once (has no parameters atm) -->
     <xacro:quadrotor_base_macro />
-    <xacro:include filename="$(find hector_sensors_description)/urdf/realsense_camera.urdf.xacro" />
-    <xacro:realsense_camera name="realsense_camera" parent="base_link">
-        <origin xyz="0.055 0.0 -0.05" rpy="0 0 0"/>
+<!--     <xacro:include filename="$(find hector_sensors_description)/urdf/realsense_camera.urdf.xacro" /> -->
+    <xacro:include filename="$(find hector_sensors_description)/urdf/hokuyo_utm30lx.urdf.xacro" />
+    <xacro:hokuyo_utm30lx name="laser0" parent="base_link" ros_topic="scan" update_rate="40" ray_count="1081" min_angle="-135" max_angle="135">
+      <origin xyz="0.0 0.0 -0.097" rpy="${M_PI} 0 0"/>
+    </xacro:hokuyo_utm30lx>
+<!--    <xacro:realsense_camera name="realsense_camera" parent="base_link">
+        <origin xyz="0.05 0.0 -0.06" rpy="0 0 0"/>
     </xacro:realsense_camera>
+ -->
+    <!-- Propiedades para simular con gazebo  -->
+    <xacro:include filename="$(find robot_auto)/urdf/kinect.urdf.xacro"/>
+    <xacro:sensor_kinect parent="base_link"/>
 </robot>

Commit message: Acercamiento robot

File: robot_auto/urdf/kinect.gazebo.xacro (robot description, xacro)
@@ -10,6 +10,6 @@
           <image>
             <format>B8G8R8</format>
-            <width>1280</width>
-            <height>720</height>
+            <width>640</width>
+            <height>480</height>
           </image>
           <clip>

File: robot_auto/urdf/kinect.urdf.xacro (robot description, xacro)
@@ -7,5 +7,5 @@
   <xacro:property name="cam_pz" value="-0.03" />
   <xacro:property name="cam_or" value="0" />
-  <xacro:property name="cam_op" value="0.30" />
+  <xacro:property name="cam_op" value="0" />
   <xacro:property name="cam_oy" value="0" />
   <xacro:property name="kinect_cam_py" value="-0.0125"/>
